File: Kicad/interrupt/interrupt.kicad_sch (KiCad schematic)
At the start: 18 parts, among them IC1 LTC1050CS8#PBF, J1 connecteur_antenne_lora, J2 Conn_GAZ, P1 Power, P2 Analog, P3 Digital, P4 Digital, P5 CONN_01X01, P6 CONN_01X01, P7 CONN_01X01, P8 CONN_01X01, Q1 IRF520

Commit message: MODIF  schéma
Connections:
- net +5V: now also J2.2 (Pin_2)
- net GAZ: now also J2.1 (Pin_1)
- net GND: now also IC1.1 (NC_1), IC1.5 (EXT_CLK_IN), IC1.8 (NC_2), J1.3 (Pin_3), J1.4 (Pin_4), J1.7 (Pin_7)
- net GNDGAZ: now also J2.3 (Pin_3)
Changed lines of the file:
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@@
     (date "lun. 30 mars 2015")
   )
+  (junction (at 120.65 125.73) (diameter 0) (color 0 0 0 0))
+  (junction (at 152.4 52.07) (diameter 0) (color 0 0 0 0))
+  (junction (at 71.12 67.31) (diameter 0) (color 0 0 0 0))
+  (junction (at 119.38 125.73) (diameter 0) (color 0 0 0 0))
+  (junction (at 151.13 52.07) (diameter 0) (color 0 0 0 0))
   (junction (at 91.44 67.31) (diameter 0) (color 0 0 0 0))
+  (junction (at 99.06 80.01) (diameter 0) (color 0 0 0 0))
   (junction (at 236.22 55.88) (diameter 1.016) (color 0 0 0 0))
-  (junction (at 99.06 80.01) (diameter 0) (color 0 0 0 0))
-  (junction (at 151.13 52.07) (diameter 0) (color 0 0 0 0))
-  (junction (at 71.12 67.31) (diameter 0) (color 0 0 0 0))
+  (junction (at 118.11 125.73) (diameter 0) (color 0 0 0 0))
   (junction (at 71.12 80.01) (diameter 0) (color 0 0 0 0))
-  (junction (at 152.4 52.07) (diameter 0) (color 0 0 0 0))
   (no_connect (at 279.4 21.59))
   (no_connect (at 274.32 21.59))
@@
     (stroke (width 0) (type dash) (color 0 0 0 0))
   )
+  (wire (pts (xy 115.57 123.19) (xy 118.11 123.19))
+    (stroke (width 0) (type default) (color 0 0 0 0))
+  )
+  (wire (pts (xy 118.11 123.19) (xy 118.11 125.73))
+    (stroke (width 0) (type default) (color 0 0 0 0))
+  )
   (wire (pts (xy 259.08 63.5) (xy 267.97 63.5))
     (stroke (width 0) (type solid) (color 0 0 0 0))
@@
     (stroke (width 0) (type solid) (color 0 0 0 0))
   )
+  (wire (pts (xy 148.59 58.42) (xy 148.59 54.61))
+    (stroke (width 0) (type default) (color 0 0 0 0))
+  )
   (wire (pts (xy 115.57 120.65) (xy 133.35 120.65))
     (stroke (width 0) (type default) (color 255 0 0 1))
@@
     (stroke (width 0) (type solid) (color 0 0 0 0))
   )
-  (wire (pts (xy 138.43 99.06) (xy 156.21 99.06))
+  (wire (pts (xy 115.57 99.06) (xy 133.35 99.06))
     (stroke (width 0) (type default) (color 0 0 0 0))
   )
@@
     (stroke (width 0) (type dash) (color 0 0 0 0))
   )
-  (wire (pts (xy 138.43 101.6) (xy 138.43 106.68))
+  (wire (pts (xy 128.27 101.6) (xy 133.35 101.6))
     (stroke (width 0) (type default) (color 0 0 0 0))
   )
@@
     (stroke (width 0) (type default) (color 0 0 0 0))
   )
+  (wire (pts (xy 115.57 115.57) (xy 119.38 115.57))
+    (stroke (width 0) (type default) (color 0 0 0 0))
+  )
+  (wire (pts (xy 119.38 115.57) (xy 119.38 125.73))
+    (stroke (width 0) (type default) (color 0 0 0 0))
+  )
   (wire (pts (xy 236.22 55.88) (xy 236.22 80.01))
     (stroke (width 0) (type solid) (color 0 0 0 0))
@@
   )
   (wire (pts (xy 99.06 80.01) (xy 151.13 80.01))
+    (stroke (width 0) (type default) (color 0 0 0 0))
+  )
+  (wire (pts (xy 115.57 113.03) (xy 120.65 113.03))
+    (stroke (width 0) (type default) (color 0 0 0 0))
+  )
+  (wire (pts (xy 120.65 113.03) (xy 120.65 125.73))
     (stroke (width 0) (type default) (color 0 0 0 0))
   )
@@
     (stroke (width 0) (type solid) (color 0 0 0 0))
   )
-  (wire (pts (xy 115.57 125.73) (xy 121.92 125.73))
+  (wire (pts (xy 118.11 125.73) (xy 119.38 125.73))
+    (stroke (width 0) (type default) (color 0 0 0 1))
+  )
+  (wire (pts (xy 115.57 125.73) (xy 118.11 125.73))
+    (stroke (width 0) (type default) (color 0 0 0 1))
+  )
+  (wire (pts (xy 120.65 125.73) (xy 125.73 125.73))
+    (stroke (width 0) (type default) (color 0 0 0 1))
+  )
+  (wire (pts (xy 119.38 125.73) (xy 120.65 125.73))
     (stroke (width 0) (type default) (color 0 0 0 1))
   )
@@
     (stroke (width 0) (type dash) (color 0 0 0 0))
   )
-  (wire (pts (xy 138.43 96.52) (xy 146.05 96.52))
+  (wire (pts (xy 125.73 96.52) (xy 133.35 96.52))
     (stroke (width 0) (type default) (color 0 0 0 0))
   )
@@
     (effects (font (size 1.524 1.524)) (justify left bottom))
   )
-  (text "connecteur pour fixer capteur de gaz\n " (at 92.71 99.06 0)
+  (text "connecteur pour fixer capteur de gaz\n " (at 91.44 95.25 0)
     (effects (font (size 1.27 1.27)) (justify left bottom))
   )
@@
     (effects (font (size 1.524 1.524)) (justify left bottom))
   )
-  (label "GAZ" (at 146.05 96.52 0)
+  (label "GAZ" (at 125.73 96.52 0)
     (effects (font (size 1.27 1.27)) (justify left bottom))
   )
@@
     (effects (font (size 1.524 1.524)) (justify left bottom))
   )
-  (label "GNDGAZ" (at 138.43 106.68 0)
+  (label "GNDGAZ" (at 128.27 101.6 0)
     (effects (font (size 1.27 1.27)) (justify left bottom))
   )
@@
     (pin "8")
   )
+  (symbol (lib_id "power:GND") (at 148.59 58.42 0) (unit 1)
+    (in_bom yes) (on_board yes) (fields_autoplaced)
+    (property "Reference" "#PWR0114" (id 0) (at 148.59 64.77 0)
+      (effects (font (size 1.27 1.27)) hide)
+    )
+    (property "Value" "GND" (id 1) (at 148.59 63.5 0))
+    (property "Footprint" "" (id 2) (at 148.59 58.42 0)
+      (effects (font (size 1.27 1.27)) hide)
+    )
+    (property "Datasheet" "" (id 3) (at 148.59 58.42 0)
+      (effects (font (size 1.27 1.27)) hide)
+    )
+    (pin "1")
+  )
   (symbol (lib_id "Device:R") (at 71.12 86.36 0) (unit 1)
     (in_bom yes) (on_board yes) (fields_autoplaced)
@@
     (pin "1")
   )
-  (symbol (lib_id "power:+5V") (at 156.21 99.06 0) (unit 1)
-    (in_bom yes) (on_board yes)
-    (property "Reference" "#PWR0101" (id 0) (at 156.21 102.87 0)
-      (effects (font (size 1.27 1.27)) hide)
-    )
-    (property "Value" "+5V" (id 1) (at 156.21 93.98 90))
-    (property "Footprint" "" (id 2) (at 156.21 99.06 0))
-    (property "Datasheet" "" (id 3) (at 156.21 99.06 0))
-    (pin "1")
-  )
-  (symbol (lib_id "power:GND") (at 121.92 125.73 0) (unit 1)
-    (in_bom yes) (on_board yes) (fields_autoplaced)
-    (property "Reference" "#PWR0108" (id 0) (at 121.92 132.08 0)
-      (effects (font (size 1.27 1.27)) hide)
-    )
-    (property "Value" "GND" (id 1) (at 121.92 130.81 0))
-    (property "Footprint" "" (id 2) (at 121.92 125.73 0)
-      (effects (font (size 1.27 1.27)) hide)
-    )
-    (property "Datasheet" "" (id 3) (at 121.92 125.73 0)
+  (symbol (lib_id "power:+5V") (at 115.57 99.06 0) (unit 1)
+    (in_bom yes) (on_board yes)
+    (property "Reference" "#PWR0101" (id 0) (at 115.57 102.87 0)
+      (effects (font (size 1.27 1.27)) hide)
+    )
+    (property "Value" "+5V" (id 1) (at 115.57 93.98 90))
+    (property "Footprint" "" (id 2) (at 115.57 99.06 0))
+    (property "Datasheet" "" (id 3) (at 115.57 99.06 0))
+    (pin "1")
+  )
+  (symbol (lib_id "power:GND") (at 125.73 125.73 0) (unit 1)
+    (in_bom yes) (on_board yes) (fields_autoplaced)
+    (property "Reference" "#PWR0108" (id 0) (at 125.73 132.08 0)
+      (effects (font (size 1.27 1.27)) hide)
+    )
+    (property "Value" "GND" (id 1) (at 125.73 130.81 0))
+    (property "Footprint" "" (id 2) (at 125.73 125.73 0)
+      (effects (font (size 1.27 1.27)) hide)
+    )
+    (property "Datasheet" "" (id 3) (at 125.73 125.73 0)
       (effects (font (size 1.27 1.27)) hide)
     )
@@
     (pin "1")
   )
+  (symbol (lib_id "power:GND") (at 148.59 46.99 90) (unit 1)
+    (in_bom yes) (on_board yes) (fields_autoplaced)
+    (property "Reference" "#PWR0112" (id 0) (at 154.94 46.99 0)
+      (effects (font (size 1.27 1.27)) hide)
+    )
+    (property "Value" "GND" (id 1) (at 152.4 46.9899 90)
+      (effects (font (size 1.27 1.27)) (justify right))
+    )
+    (property "Footprint" "" (id 2) (at 148.59 46.99 0)
+      (effects (font (size 1.27 1.27)) hide)
+    )
+    (property "Datasheet" "" (id 3) (at 148.59 46.99 0)
+      (effects (font (size 1.27 1.27)) hide)
+    )
+    (pin "1")
+  )
   (symbol (lib_id "Device:R") (at 91.44 73.66 0) (unit 1)
     (in_bom yes) (on_board yes) (fields_autoplaced)
@@
     (pin "1")
   )
+  (symbol (lib_id "power:GND") (at 113.03 46.99 270) (unit 1)
+    (in_bom yes) (on_board yes) (fields_autoplaced)
+    (property "Reference" "#PWR0113" (id 0) (at 106.68 46.99 0)
+      (effects (font (size 1.27 1.27)) hide)
+    )
+    (property "Value" "GND" (id 1) (at 109.22 46.9899 90)
+      (effects (font (size 1.27 1.27)) (justify right))
+    )
+    (property "Footprint" "" (id 2) (at 113.03 46.99 0)
+      (effects (font (size 1.27 1.27)) hide)
+    )
+    (property "Datasheet" "" (id 3) (at 113.03 46.99 0)
+      (effects (font (size 1.27 1.27)) hide)
+    )
+    (pin "1")
+  )
   (sheet_instances
     (path "/" (page "1"))
@@
       (reference "#PWR0111") (unit 1) (value "GND") (footprint "")
     )
+    (path "/cfed5c4e-149f-45c5-874a-d4efe242083a"
+      (reference "#PWR0112") (unit 1) (value "GND") (footprint "")
+    )
+    (path "/ff14d0d7-f586-47b8-af56-707d6fdbcef9"
+      (reference "#PWR0113") (unit 1) (value "GND") (footprint "")
+    )
+    (path "/5302655e-adcd-494d-9861-53f4df5616e5"
+      (reference "#PWR0114") (unit 1) (value "GND") (footprint "")
+    )
     (path "/15512f16-8e00-43a9-a6a5-92f2a94616db"

Commit message: modification schéma kicad
Parts:
- removed C1: 100u, Capacitor_THT:C_Radial_D4.0mm_H5.0mm_P1.50mm, symbol Device:C
- removed J1: connecteur_antenne_lora, Connector_JST:JST_EH_B8B-EH-A_1x08_P2.50mm_Vertical, symbol Connector:Conn_01x08_Male
- removed J2: Conn_GAZ, Connector_JST:JST_XH_B3B-XH-A_1x03_P2.50mm_Vertical, symbol Connector:Conn_01x03_Female
- added C1: C_Polarized, Capacitor_THT:CP_Radial_D4.0mm_P2.00mm, symbol Device:C_Polarized
- added R2: 1M, Resistor_THT:R_Axial_DIN0204_L3.6mm_D1.6mm_P5.08mm_Horizontal, symbol Device:R
- renumbered R2 to R3
Connections:
- net GNDGAZ is gone; now on net VNGAZ: Q1.2
- net +3V3: no longer IC1.7 (V+)
- net +5V: now also IC1.7 (V+), C1.1
- net VAOP: now also R2.1; no longer IC1.3 (+IN), R4.2, R5.1
- net at R3.1: now also IC1.3 (+IN), R4.2, R5.1; no longer R1.2
- net GAZ renamed VNGAZ
- new net: C1.2, R1.2, R2.2
Other:
- note removed: "connecteur pour fixer antenne lora"
- note removed: "connecteur pour fixer capteur de gaz"
- moved on the sheet: R3

Commit message: mis
Parts:
- added Cd1, Cd3, Cd4: 100n, symbol Device:C
- added Cd2: 1u, symbol Device:C
- added ICd1: LTC1050CS8#PBF, ltc 1050:PDIP-8_N, symbol LTC1050CS8#PBF:LTC1050CS8#PBF
- added Rd1: 10k, symbol Device:R
- added Rd2, Rd4: 100k, symbol Device:R
- added Rd3, Rd5: 1k, symbol Device:R
Connections:
- net +5V: now also Cd4.1, ICd1.7 (V+)
- net GND: now also Cd1.2, Cd3.2, Cd4.2, ICd1.4 (V-), Rd2.2, Rd3.2; no longer IC1.1 (NC_1), IC1.5 (EXT_CLK_IN), IC1.8 (NC_2)
- net VNGAZ renamed Data_Gaz
- net Data_Gaz: no longer Q1.2
- new net: Cd2.1, ICd1.2 (-IN), Rd3.1, Rd4.1
- new net: Cd1.1, ICd1.3 (+IN), Rd1.2, Rd2.1
- new net: Cd2.2, ICd1.6 (OUT), Rd4.2, Rd5.1
- new net: Cd3.1, Rd5.2
- new net GND_Gaz: Q1.2
- no-connect marks 5 -> 11
Other:
- moved on the sheet: C1, IC1, Q1, R1, R2, R3, R4, R5, R6

Commit message: maj
Parts:
- added U?: GAZ_TO_5, symbol Gaz_sensor:GAZ_TO_5
Other:
- moved on the sheet: Cd1, Cd2, Cd3, Cd4, ICd1, Rd1, Rd2, Rd3, Rd4, Rd5

Commit message: maj
Parts:
- removed U?: GAZ_TO_5, symbol Gaz_sensor:GAZ_TO_5
- added U?: GAZ_TO_5, symbol Gaz_sensor:GAZ_TO_5
Connections:
- net +5V: now also U?.7 (R_Sens_2_IN)
- no-connect marks 11 -> 13

Commit message: maj
Parts:
- Cd1, Cd2, Cd3, Cd4: footprint (none) -> Capacitor_THT:C_Radial_D4.0mm_H5.0mm_P1.50mm
- Rd1, Rd2, Rd3, Rd4, Rd5: footprint (none) -> Resistor_THT:R_Axial_DIN0204_L3.6mm_D1.6mm_P5.08mm_Horizontal
- U1: renamed from U?; footprint (none) -> GAZ_foot_print:GAZ_TO-5

Commit message: maj
Parts:
- added Ral: R, symbol Device:R
Connections:
- net +5V: now also U1.2 (R_Sens_1_IN), U1.3 (R_Poly_IN); no longer U1.7 (R_Sens_2_IN)
- net GND: now also U1.6 (R_ALU_OUT)
- net at Rd1.1: now also U1.4 (R_Sens_1_OUT)
- net at U1.1 (R_ALU_IN): now also Ral.2
- new net +3V0: Ral.1
- no-connect marks 13 -> 15
Other:
- moved on the sheet: U1

Commit message: maj
Parts:
- added J1: Conn_LORA, Connector_PinSocket_2.54mm:PinSocket_1x08_P2.54mm_Vertical, symbol Connector:Conn_01x08_Female
- Ral1: renamed from Ral; footprint (none) -> Resistor_THT:R_Axial_DIN0204_L3.6mm_D1.6mm_P5.08mm_Horizontal
Connections:
- net +3V0 is gone; now on net +3V3: Ral1.1
- net A0 is gone; now on net DATA_Sensor: P2.1 (Pin_1)
- net +3V3: now also J1.6 (Pin_6)
- net GND: now also J1.8 (Pin_8)
- net GND_Gaz: now also U1.8 (R_Poly_OUT)
- net RST: now also J1.5 (Pin_5)
- net RX: now also J1.2 (Pin_2)
- net TX: now also J1.1 (Pin_1)
- net DATA_Sensor: now reaches Cd3.1, Rd5.2
- new net CTS: J1.3 (Pin_3)
- new net RTS: J1.4 (Pin_4)
- new net VIN_L: J1.7 (Pin_7)
Other:
- moved on the sheet: Ral1
