File: Kicad/interrupt/interrupt.kicad_sch (KiCad schematic)
At the start: 30 parts, among them IC1 LTC1050CS8#PBF, J1 Conn_LORA, P1 Power, P2 Analog, P3 Digital, P4 Digital, P5 CONN_01X01, P6 CONN_01X01, P7 CONN_01X01, P8 CONN_01X01, Q1 IRF520, U1 GAZ_TO_5

Commit message: maj
Parts:
- Q1: footprint IRF520:TO270P460X1020X2008-3P -> KiCadIRF:TO254P465X1024X2050-3P
Connections:
- net A2 is gone; now on net R_Alu_Temp: P2.3 (Pin_3)
- net R_Alu_Temp: now reaches Ral1.2, U1.1 (R_ALU_IN)
Other:
- moved on the sheet: Ral1
Changed lines of the file:
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@@
     (date "lun. 30 mars 2015")
   )
+  (junction (at 236.22 55.88) (diameter 1.016) (color 0 0 0 0))
   (junction (at 191.77 101.6) (diameter 0) (color 0 0 0 0))
+  (junction (at 200.66 125.73) (diameter 0) (color 0 0 0 0))
+  (junction (at 43.18 43.18) (diameter 0) (color 0 0 0 0))
+  (junction (at 120.65 144.78) (diameter 0) (color 0 0 0 0))
+  (junction (at 191.77 125.73) (diameter 0) (color 0 0 0 0))
+  (junction (at 27.94 43.18) (diameter 0) (color 0 0 0 0))
+  (junction (at 27.94 55.88) (diameter 0) (color 0 0 0 0))
+  (junction (at 120.65 125.73) (diameter 0) (color 0 0 0 0))
+  (junction (at 133.35 123.19) (diameter 0) (color 0 0 0 0))
+  (junction (at 220.98 96.52) (diameter 0) (color 0 0 0 0))
+  (junction (at 220.98 125.73) (diameter 0) (color 0 0 0 0))
+  (junction (at 38.1 102.87) (diameter 0) (color 0 0 0 0))
+  (junction (at 107.95 27.94) (diameter 0) (color 0 0 0 0))
+  (junction (at 147.32 144.78) (diameter 0) (color 0 0 0 0))
+  (junction (at 220.98 144.78) (diameter 0) (color 0 0 0 0))
+  (junction (at 109.22 125.73) (diameter 0) (color 0 0 0 0))
+  (junction (at 110.49 27.94) (diameter 0) (color 0 0 0 0))
+  (junction (at 55.88 55.88) (diameter 0) (color 0 0 0 0))
   (junction (at 133.35 144.78) (diameter 0) (color 0 0 0 0))
-  (junction (at 133.35 123.19) (diameter 0) (color 0 0 0 0))
-  (junction (at 110.49 27.94) (diameter 0) (color 0 0 0 0))
-  (junction (at 147.32 144.78) (diameter 0) (color 0 0 0 0))
-  (junction (at 191.77 125.73) (diameter 0) (color 0 0 0 0))
-  (junction (at 107.95 27.94) (diameter 0) (color 0 0 0 0))
-  (junction (at 220.98 125.73) (diameter 0) (color 0 0 0 0))
-  (junction (at 220.98 96.52) (diameter 0) (color 0 0 0 0))
-  (junction (at 27.94 43.18) (diameter 0) (color 0 0 0 0))
-  (junction (at 220.98 144.78) (diameter 0) (color 0 0 0 0))
-  (junction (at 27.94 55.88) (diameter 0) (color 0 0 0 0))
-  (junction (at 109.22 125.73) (diameter 0) (color 0 0 0 0))
-  (junction (at 120.65 125.73) (diameter 0) (color 0 0 0 0))
-  (junction (at 43.18 43.18) (diameter 0) (color 0 0 0 0))
-  (junction (at 236.22 55.88) (diameter 1.016) (color 0 0 0 0))
-  (junction (at 200.66 125.73) (diameter 0) (color 0 0 0 0))
-  (junction (at 55.88 55.88) (diameter 0) (color 0 0 0 0))
-  (junction (at 120.65 144.78) (diameter 0) (color 0 0 0 0))
+  (no_connect (at 182.88 128.27))
   (no_connect (at 182.88 120.65))
-  (no_connect (at 182.88 128.27))
   (no_connect (at 147.32 120.65))
   (no_connect (at 105.41 22.86))
@@
     (stroke (width 0) (type default) (color 0 0 0 0))
   )
+  (wire (pts (xy 38.1 100.33) (xy 38.1 102.87))
+    (stroke (width 0) (type default) (color 0 0 0 0))
+  )
   (wire (pts (xy 238.76 71.12) (xy 226.06 71.12))
     (stroke (width 0) (type solid) (color 0 0 0 0))
@@
     (stroke (width 0) (type default) (color 0 0 0 0))
   )
+  (wire (pts (xy 200.66 106.68) (xy 200.66 101.6))
+    (stroke (width 0) (type default) (color 0 0 0 0))
+  )
   (wire (pts (xy 191.77 101.6) (xy 200.66 101.6))
-    (stroke (width 0) (type default) (color 0 0 0 0))
-  )
-  (wire (pts (xy 200.66 106.68) (xy 200.66 101.6))
     (stroke (width 0) (type default) (color 0 0 0 0))
   )
@@
     (stroke (width 0) (type solid) (color 0 0 0 0))
   )
+  (wire (pts (xy 110.49 13.97) (xy 43.18 13.97))
+    (stroke (width 0) (type default) (color 0 0 0 0))
+  )
+  (wire (pts (xy 43.18 13.97) (xy 43.18 16.51))
+    (stroke (width 0) (type default) (color 0 0 0 0))
+  )
   (wire (pts (xy 110.49 27.94) (xy 110.49 13.97))
-    (stroke (width 0) (type default) (color 0 0 0 0))
-  )
-  (wire (pts (xy 110.49 13.97) (xy 43.18 13.97))
-    (stroke (width 0) (type default) (color 0 0 0 0))
-  )
-  (wire (pts (xy 43.18 13.97) (xy 43.18 16.51))
     (stroke (width 0) (type default) (color 0 0 0 0))
   )
@@
     (stroke (width 0) (type default) (color 0 0 0 0))
   )
-  (wire (pts (xy 38.1 91.44) (xy 38.1 95.25))
+  (wire (pts (xy 38.1 91.44) (xy 38.1 92.71))
     (stroke (width 0) (type default) (color 0 0 0 0))
   )
@@
     (stroke (width 0) (type default) (color 0 0 0 0))
   )
+  (wire (pts (xy 133.35 144.78) (xy 147.32 144.78))
+    (stroke (width 0) (type default) (color 0 0 0 0))
+  )
+  (wire (pts (xy 120.65 144.78) (xy 133.35 144.78))
+    (stroke (width 0) (type default) (color 0 0 0 0))
+  )
   (wire (pts (xy 109.22 144.78) (xy 120.65 144.78))
-    (stroke (width 0) (type default) (color 0 0 0 0))
-  )
-  (wire (pts (xy 120.65 144.78) (xy 133.35 144.78))
-    (stroke (width 0) (type default) (color 0 0 0 0))
-  )
-  (wire (pts (xy 133.35 144.78) (xy 147.32 144.78))
     (stroke (width 0) (type default) (color 0 0 0 0))
   )
@@
     (stroke (width 0) (type solid) (color 0 0 0 0))
   )
+  (wire (pts (xy 191.77 125.73) (xy 200.66 125.73))
+    (stroke (width 0) (type default) (color 0 0 0 0))
+  )
   (wire (pts (xy 182.88 125.73) (xy 191.77 125.73))
     (stroke (width 0) (type default) (color 0 0 0 0))
   )
-  (wire (pts (xy 191.77 125.73) (xy 200.66 125.73))
-    (stroke (width 0) (type default) (color 0 0 0 0))
-  )
   (wire (pts (xy 200.66 125.73) (xy 208.28 125.73))
     (stroke (width 0) (type default) (color 0 0 0 0))
@@
     (stroke (width 0) (type default) (color 0 0 0 0))
   )
+  (wire (pts (xy 43.18 43.18) (xy 48.26 43.18))
+    (stroke (width 0) (type default) (color 0 0 0 0))
+  )
   (wire (pts (xy 41.91 43.18) (xy 43.18 43.18))
-    (stroke (width 0) (type default) (color 0 0 0 0))
-  )
-  (wire (pts (xy 43.18 43.18) (xy 48.26 43.18))
     (stroke (width 0) (type default) (color 0 0 0 0))
   )
@@
     (stroke (width 0) (type solid) (color 0 0 0 0))
   )
+  (wire (pts (xy 220.98 125.73) (xy 220.98 128.27))
+    (stroke (width 0) (type default) (color 0 0 0 0))
+  )
   (wire (pts (xy 215.9 125.73) (xy 220.98 125.73))
-    (stroke (width 0) (type default) (color 0 0 0 0))
-  )
-  (wire (pts (xy 220.98 125.73) (xy 220.98 128.27))
     (stroke (width 0) (type default) (color 0 0 0 0))
   )
@@
     (stroke (width 0) (type default) (color 0 0 0 0))
   )
+  (wire (pts (xy 110.49 27.94) (xy 114.3 27.94))
+    (stroke (width 0) (type default) (color 0 0 0 0))
+  )
   (wire (pts (xy 107.95 27.94) (xy 110.49 27.94))
-    (stroke (width 0) (type default) (color 0 0 0 0))
-  )
-  (wire (pts (xy 110.49 27.94) (xy 114.3 27.94))
     (stroke (width 0) (type default) (color 0 0 0 0))
   )
@@
     (stroke (width 0) (type default) (color 0 0 0 0))
   )
+  (wire (pts (xy 33.02 102.87) (xy 38.1 102.87))
+    (stroke (width 0) (type default) (color 0 0 0 0))
+  )
+  (wire (pts (xy 186.69 123.19) (xy 186.69 96.52))
+    (stroke (width 0) (type default) (color 0 0 0 0))
+  )
   (wire (pts (xy 182.88 123.19) (xy 186.69 123.19))
-    (stroke (width 0) (type default) (color 0 0 0 0))
-  )
-  (wire (pts (xy 186.69 123.19) (xy 186.69 96.52))
     (stroke (width 0) (type default) (color 0 0 0 0))
   )
@@
     (effects (font (size 1.27 1.27)) (justify left bottom))
   )
+  (label "R_Alu_Temp" (at 33.02 102.87 180)
+    (effects (font (size 1.27 1.27)) (justify right bottom))
+  )
   (label "VIN_L" (at 30.48 171.45 0)
     (effects (font (size 1.27 1.27)) (justify left bottom))
@@
     (effects (font (size 1.524 1.524)) (justify left bottom))
   )
-  (label "A2" (at 226.06 68.58 0)
+  (label "R_Alu_Temp" (at 226.06 68.58 0)
     (effects (font (size 1.524 1.524)) (justify left bottom))
   )
@@
       (effects (font (size 1.27 1.27)) (justify left))
     )
-    (property "Footprint" "IRF520:TO270P460X1020X2008-3P" (id 2) (at 139.7 40.64 0)
+    (property "Footprint" "KiCadIRF:TO254P465X1024X2050-3P" (id 2) (at 139.7 40.64 0)
       (effects (font (size 1.27 1.27)) (justify left) hide)
     )
@@
     (pin "1")
   )
-  (symbol (lib_id "Device:R") (at 38.1 99.06 0) (unit 1)
-    (in_bom yes) (on_board yes) (fields_autoplaced)
-    (property "Reference" "Ral1" (id 0) (at 40.64 97.7899 0)
-      (effects (font (size 1.27 1.27)) (justify left))
-    )
-    (property "Value" "R" (id 1) (at 40.64 100.3299 0)
-      (effects (font (size 1.27 1.27)) (justify left))
-    )
-    (property "Footprint" "Resistor_THT:R_Axial_DIN0204_L3.6mm_D1.6mm_P5.08mm_Horizontal" (id 2) (at 36.322 99.06 90)
-      (effects (font (size 1.27 1.27)) hide)
-    )
-    (property "Datasheet" "~" (id 3) (at 38.1 99.06 0)
+  (symbol (lib_id "Device:R") (at 38.1 96.52 0) (unit 1)
+    (in_bom yes) (on_board yes) (fields_autoplaced)
+    (property "Reference" "Ral1" (id 0) (at 40.64 95.2499 0)
+      (effects (font (size 1.27 1.27)) (justify left))
+    )
+    (property "Value" "R" (id 1) (at 40.64 97.7899 0)
+      (effects (font (size 1.27 1.27)) (justify left))
+    )
+    (property "Footprint" "Resistor_THT:R_Axial_DIN0204_L3.6mm_D1.6mm_P5.08mm_Horizontal" (id 2) (at 36.322 96.52 90)
+      (effects (font (size 1.27 1.27)) hide)
+    )
+    (property "Datasheet" "~" (id 3) (at 38.1 96.52 0)
       (effects (font (size 1.27 1.27)) hide)
     )
@@
     )
     (path "/5e2f2c9c-430a-4909-b481-b198cf5a3f05"
-      (reference "Q1") (unit 1) (value "IRF520") (footprint "IRF520:TO270P460X1020X2008-3P")
+      (reference "Q1") (unit 1) (value "IRF520") (footprint "KiCadIRF:TO254P465X1024X2050-3P")
     )
     (path "/0fb4e2ba-9e00-4f1b-8b29-934a5a1ace04"

Commit message: maj
Other:
- company: (none) -> INSA 
- title: (none) -> Projet MOSH
Changed lines of the file:
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@@
   (paper "A4")
   (title_block
+    (title "Projet MOSH")
     (date "lun. 30 mars 2015")
-  )
+    (rev "1.0")
+    (company "INSA ")
+    (comment 1 "KHALED LEON GENEAU ")
+    (comment 2 "wkhaled@insa-toulouse.fr")
+  )
+  (junction (at 220.98 144.78) (diameter 0) (color 0 0 0 0))
   (junction (at 236.22 55.88) (diameter 1.016) (color 0 0 0 0))
+  (junction (at 109.22 125.73) (diameter 0) (color 0 0 0 0))
+  (junction (at 147.32 144.78) (diameter 0) (color 0 0 0 0))
+  (junction (at 55.88 55.88) (diameter 0) (color 0 0 0 0))
+  (junction (at 191.77 125.73) (diameter 0) (color 0 0 0 0))
+  (junction (at 133.35 123.19) (diameter 0) (color 0 0 0 0))
+  (junction (at 220.98 125.73) (diameter 0) (color 0 0 0 0))
+  (junction (at 107.95 27.94) (diameter 0) (color 0 0 0 0))
+  (junction (at 200.66 125.73) (diameter 0) (color 0 0 0 0))
+  (junction (at 120.65 125.73) (diameter 0) (color 0 0 0 0))
+  (junction (at 27.94 55.88) (diameter 0) (color 0 0 0 0))
+  (junction (at 27.94 43.18) (diameter 0) (color 0 0 0 0))
+  (junction (at 120.65 144.78) (diameter 0) (color 0 0 0 0))
+  (junction (at 133.35 144.78) (diameter 0) (color 0 0 0 0))
+  (junction (at 220.98 96.52) (diameter 0) (color 0 0 0 0))
+  (junction (at 38.1 102.87) (diameter 0) (color 0 0 0 0))
+  (junction (at 43.18 43.18) (diameter 0) (color 0 0 0 0))
+  (junction (at 110.49 27.94) (diameter 0) (color 0 0 0 0))
   (junction (at 191.77 101.6) (diameter 0) (color 0 0 0 0))
-  (junction (at 200.66 125.73) (diameter 0) (color 0 0 0 0))
-  (junction (at 43.18 43.18) (diameter 0) (color 0 0 0 0))
-  (junction (at 120.65 144.78) (diameter 0) (color 0 0 0 0))
-  (junction (at 191.77 125.73) (diameter 0) (color 0 0 0 0))
-  (junction (at 27.94 43.18) (diameter 0) (color 0 0 0 0))
-  (junction (at 27.94 55.88) (diameter 0) (color 0 0 0 0))
-  (junction (at 120.65 125.73) (diameter 0) (color 0 0 0 0))
-  (junction (at 133.35 123.19) (diameter 0) (color 0 0 0 0))
-  (junction (at 220.98 96.52) (diameter 0) (color 0 0 0 0))
-  (junction (at 220.98 125.73) (diameter 0) (color 0 0 0 0))
-  (junction (at 38.1 102.87) (diameter 0) (color 0 0 0 0))
-  (junction (at 107.95 27.94) (diameter 0) (color 0 0 0 0))
-  (junction (at 147.32 144.78) (diameter 0) (color 0 0 0 0))
-  (junction (at 220.98 144.78) (diameter 0) (color 0 0 0 0))
-  (junction (at 109.22 125.73) (diameter 0) (color 0 0 0 0))
-  (junction (at 110.49 27.94) (diameter 0) (color 0 0 0 0))
-  (junction (at 55.88 55.88) (diameter 0) (color 0 0 0 0))
-  (junction (at 133.35 144.78) (diameter 0) (color 0 0 0 0))
+  (no_connect (at 69.85 22.86))
+  (no_connect (at 105.41 34.29))
+  (no_connect (at 105.41 22.86))
   (no_connect (at 182.88 128.27))
   (no_connect (at 182.88 120.65))
   (no_connect (at 147.32 120.65))
-  (no_connect (at 105.41 22.86))
-  (no_connect (at 105.41 34.29))
-  (no_connect (at 69.85 22.86))
   (no_connect (at 279.4 21.59))
   (no_connect (at 274.32 21.59))
+  (no_connect (at 73.66 119.38))
   (no_connect (at 38.1 119.38))
-  (no_connect (at 73.66 119.38))
   (no_connect (at 276.86 21.59))
   (no_connect (at 73.66 116.84))
@@
     (stroke (width 0) (type default) (color 0 0 0 0))
   )
+  (wire (pts (xy 31.75 125.73) (xy 96.52 125.73))
+    (stroke (width 0) (type default) (color 0 0 0 0))
+  )
   (wire (pts (xy 109.22 125.73) (xy 120.65 125.73))
     (stroke (width 0) (type default) (color 0 0 0 0))
@@
   )
   (wire (pts (xy 120.65 125.73) (xy 147.32 125.73))
-    (stroke (width 0) (type default) (color 0 0 0 0))
-  )
-  (wire (pts (xy 31.75 125.73) (xy 96.52 125.73))
     (stroke (width 0) (type default) (color 0 0 0 0))
   )
@@
     (stroke (width 0) (type default) (color 0 0 0 0))
   )
+  (wire (pts (xy 133.35 123.19) (xy 133.35 133.35))
+    (stroke (width 0) (type default) (color 0 0 0 0))
+  )
   (wire (pts (xy 147.32 123.19) (xy 133.35 123.19))
-    (stroke (width 0) (type default) (color 0 0 0 0))
-  )
-  (wire (pts (xy 133.35 123.19) (xy 133.35 133.35))
     (stroke (width 0) (type default) (color 0 0 0 0))
   )
@@
     (stroke (width 0) (type solid) (color 0 0 0 0))
   )
+  (wire (pts (xy 200.66 125.73) (xy 208.28 125.73))
+    (stroke (width 0) (type default) (color 0 0 0 0))
+  )
   (wire (pts (xy 191.77 125.73) (xy 200.66 125.73))
     (stroke (width 0) (type default) (color 0 0 0 0))
@@
     (stroke (width 0) (type default) (color 0 0 0 0))
   )
-  (wire (pts (xy 200.66 125.73) (xy 208.28 125.73))
-    (stroke (width 0) (type default) (color 0 0 0 0))
-  )
   (wire (pts (xy 48.26 25.4) (xy 69.85 25.4))
     (stroke (width 0) (type default) (color 0 0 0 0))
   )
+  (wire (pts (xy 55.88 27.94) (xy 55.88 55.88))
+    (stroke (width 0) (type default) (color 0 0 0 0))
+  )
   (wire (pts (xy 55.88 55.88) (xy 27.94 55.88))
-    (stroke (width 0) (type default) (color 0 0 0 0))
-  )
-  (wire (pts (xy 55.88 27.94) (xy 55.88 55.88))
     (stroke (width 0) (type default) (color 0 0 0 0))
   )
@@
     (stroke (width 0) (type solid) (color 0 0 0 0))
   )
+  (wire (pts (xy 220.98 125.73) (xy 236.22 125.73))
+    (stroke (width 0) (type default) (color 0 0 0 0))
+  )
   (wire (pts (xy 220.98 125.73) (xy 220.98 128.27))
     (stroke (width 0) (type default) (color 0 0 0 0))
   )
   (wire (pts (xy 215.9 125.73) (xy 220.98 125.73))
-    (stroke (width 0) (type default) (color 0 0 0 0))
-  )
-  (wire (pts (xy 220.98 125.73) (xy 236.22 125.73))
     (stroke (width 0) (type default) (color 0 0 0 0))
   )
@@
     (stroke (width 0) (type default) (color 0 0 0 0))
   )
+  (wire (pts (xy 220.98 96.52) (xy 220.98 101.6))
+    (stroke (width 0) (type default) (color 0 0 0 0))
+  )
+  (wire (pts (xy 186.69 96.52) (xy 220.98 96.52))
+    (stroke (width 0) (type default) (color 0 0 0 0))
+  )
+  (wire (pts (xy 182.88 123.19) (xy 186.69 123.19))
+    (stroke (width 0) (type default) (color 0 0 0 0))
+  )
   (wire (pts (xy 186.69 123.19) (xy 186.69 96.52))
     (stroke (width 0) (type default) (color 0 0 0 0))
   )
-  (wire (pts (xy 182.88 123.19) (xy 186.69 123.19))
-    (stroke (width 0) (type default) (color 0 0 0 0))
-  )
-  (wire (pts (xy 186.69 96.52) (xy 220.98 96.52))
-    (stroke (width 0) (type default) (color 0 0 0 0))
-  )
-  (wire (pts (xy 220.98 96.52) (xy 220.98 101.6))
-    (stroke (width 0) (type default) (color 0 0 0 0))
-  )
