File: Kicad/interrupt/interrupt.kicad_pcb (KiCad board)
At the start: 2 copper layers, 68.6 x 53.3 mm, 18 parts, among them IC1 LTC1050CS8#PBF, J1 connecteur_antenne_lora, J2 Conn_GAZ, P1 Power, P2 Analog, P3 Digital, P4 Digital, P5 CONN_01X01, P6 CONN_01X01, P7 CONN_01X01, P8 CONN_01X01, Q1 IRF520

Commit message: MODIF  schéma
Connections:
- IC1 pad 1: unconnected-(IC1-Pad1) -> GND
- IC1 pad 5: unconnected-(IC1-Pad5) -> GND
- IC1 pad 8: unconnected-(IC1-Pad8) -> GND
- J1 pad 3: unconnected-(J1-Pad3) -> GND
- J1 pad 4: unconnected-(J1-Pad4) -> GND
- J1 pad 7: unconnected-(J1-Pad7) -> GND
- J2 pad 1: unconnected-(J2-Pad1) -> /GAZ
- J2 pad 2: unconnected-(J2-Pad2) -> +5V
- J2 pad 3: unconnected-(J2-Pad3) -> /GNDGAZ

Commit message: maj
Routing:
- net /TX: track 0.00 -> 27.3 mm
- added copper zone on B.Cu, net GND
Changed lines of the file:
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@@
     (effects (font (size 1 1) (thickness 0.15)))
   )
+  (segment (start 133.718 91.43) (end 141.963 83.185) (width 0.25) (layer "B.Cu") (net 22))
+  (segment (start 141.963 83.185) (end 147.828 83.185) (width 0.25) (layer "B.Cu") (net 22))
+  (segment (start 147.828 83.185) (end 149.098 81.915) (width 0.25) (layer "B.Cu") (net 22))
+  (segment (start 147.574 76.581) (end 147.574 75.565) (width 0.25) (layer "B.Cu") (net 22))
+  (segment (start 149.098 78.105) (end 147.574 76.581) (width 0.25) (layer "B.Cu") (net 22))
+  (segment (start 133.718 92.405) (end 133.718 91.43) (width 0.25) (layer "B.Cu") (net 22))
+  (segment (start 149.098 81.915) (end 149.098 78.105) (width 0.25) (layer "B.Cu") (net 22))
+  (zone (net 4) (net_name "GND") (layer "B.Cu") (hatch edge 0.508)
+    (connect_pads (clearance 0.508))
+    (min_thickness 0.254) (filled_areas_thickness no)
+    (fill (thermal_gap 0.508) (thermal_bridge_width 0.508))
+    (polygon
+      (pts
+        (xy 182.118 127.635)
+        (xy 109.728 127.635)
+        (xy 108.458 102.235)
+        (xy 108.458 73.025)
+        (xy 179.578 71.755)
+      )
+    )
+  )
 )

Commit message: maj
Parts:
- removed J2: Conn_GAZ, Connector_JST:JST_XH_B3B-XH-A_1x03_P2.50mm_Vertical
- added Cd1: 100n, Capacitor_THT:C_Radial_D4.0mm_H5.0mm_P1.50mm, F.Cu at (158.8, 101.6)
- added Cd2: 1u, Capacitor_THT:C_Radial_D4.0mm_H5.0mm_P1.50mm, F.Cu at (164.4, 104.0)
- added Cd3: 100n, Capacitor_THT:C_Radial_D4.0mm_H5.0mm_P1.50mm, F.Cu at (154.4, 107.1)
- added Cd4: 100n, Capacitor_THT:C_Radial_D4.0mm_H5.0mm_P1.50mm, F.Cu at (143.4, 118.1)
- added ICd1: LTC1050CS8#PBF, ltc 1050:PDIP-8_N, F.Cu at (165.6, 111.3)
- added R2: 1M, Resistor_THT:R_Axial_DIN0204_L3.6mm_D1.6mm_P5.08mm_Horizontal, F.Cu at (177.6, 96.9)
- added Ral1: R, Resistor_THT:R_Axial_DIN0204_L3.6mm_D1.6mm_P5.08mm_Horizontal, F.Cu at (169.5, 98.3)
- added Rd1: 10k, Resistor_THT:R_Axial_DIN0204_L3.6mm_D1.6mm_P5.08mm_Horizontal, F.Cu at (173.0, 107.7)
- added Rd2: 100k, Resistor_THT:R_Axial_DIN0204_L3.6mm_D1.6mm_P5.08mm_Horizontal, F.Cu at (163.0, 108.3)
- added Rd3: 1k, Resistor_THT:R_Axial_DIN0204_L3.6mm_D1.6mm_P5.08mm_Horizontal, F.Cu at (173.0, 104.6)
- added Rd4: 100k, Resistor_THT:R_Axial_DIN0204_L3.6mm_D1.6mm_P5.08mm_Horizontal, F.Cu at (152.0, 119.3)
- added Rd5: 1k, Resistor_THT:R_Axial_DIN0204_L3.6mm_D1.6mm_P5.08mm_Horizontal, F.Cu at (173.0, 101.4)
- added U1: GAZ_TO_5, GAZ_foot_print:GAZ_TO-5, F.Cu at (138.1, 117.9)
- C1: value 100u -> C_Polarized; footprint Capacitor_THT:C_Radial_D4.0mm_H5.0mm_P1.50mm -> Capacitor_THT:CP_Radial_D4.0mm_P2.00mm
- J1: value connecteur_antenne_lora -> Conn_LORA; footprint Connector_JST:JST_EH_B8B-EH-A_1x08_P2.50mm_Vertical -> Connector_PinSocket_2.54mm:PinSocket_1x08_P2.54mm_Vertical
- moved J1 50.3 mm to (176.7, 118.5), turned to 180 degrees
- moved Q1 19.0 mm to (117.2, 109.4)
- moved C1 11.7 mm to (151.6, 114.9), turned to 180 degrees
- renumbered R2 to R3
Connections:
- IC1 pad 1: GND -> unconnected-(IC1-Pad1)
- IC1 pad 3: /VAOP -> Net-(IC1-Pad3)
- IC1 pad 5: GND -> unconnected-(IC1-Pad5)
- IC1 pad 7: +3V3 -> +5V
- IC1 pad 8: GND -> unconnected-(IC1-Pad8)
- J1 pad 3: GND -> /CTS
- J1 pad 4: GND -> /RTS
- J1 pad 7: GND -> /VIN_L
- P2 pad 1: /A0 -> /DATA_Sensor
- P2 pad 2: /GAZ -> /Data_Gaz
- Q1 pad 2: /GNDGAZ -> /GND_Gaz
- R3 pad 1: Net-(C1-Pad2) -> Net-(IC1-Pad3)
- R4 pad 2: /VAOP -> Net-(IC1-Pad3)
- R5 pad 1: /VAOP -> Net-(IC1-Pad3)
Routing:
- net /TX: track 27.3 -> 1.99 mm

Commit message: maj
Parts:
- Q1: footprint IRF520:TO270P460X1020X2008-3P -> KiCadIRF:TO254P465X1024X2050-3P
- moved R2 39.6 mm to (141.5, 80.6)
- moved R1 32.0 mm to (127.5, 80.6)
- moved Ral1 26.0 mm to (150.4, 80.6)
- moved R3 23.0 mm to (140.2, 85.7)
- moved U1 22.5 mm to (122.8, 101.4)
- moved IC1 19.8 mm to (135.1, 93.3)
- moved Cd2 16.4 mm to (154.5, 90.9)
- moved Cd1 16.4 mm to (148.9, 88.5)
- moved Rd2 16.4 mm to (153.1, 95.2)
- moved Q1 14.2 mm to (128.8, 117.5)
- moved R4 8.61 mm to (140.2, 102.2)
- moved Rd3 6.86 mm to (168.1, 99.7)
- moved Rd1 6.86 mm to (168.1, 102.8)
- moved Rd5 6.86 mm to (168.1, 96.5)
- moved ICd1 5.75 mm to (160.5, 108.6)
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Routing:
- net GND: track 0.00 -> 172.8 mm
- net +5V: track 0.00 -> 166.8 mm
- net Net-(IC1-Pad3): track 0.00 -> 99.2 mm
- net Net-(Cd2-Pad1): track 0.00 -> 70.3 mm
- net Net-(Cd2-Pad2): track 0.00 -> 65.2 mm
- net /VAOP: track 0.00 -> 62.3 mm
- net /TX: track 1.99 -> 61.5 mm, vias 0 -> 1
- net Net-(C1-Pad2): track 0.00 -> 56.4 mm, vias 0 -> 2
- net /RST: track 0.00 -> 52.8 mm, vias 0 -> 1
- net +3V3: track 0.00 -> 42.0 mm, vias 0 -> 1
- net Net-(Cd1-Pad1): track 0.00 -> 38.6 mm
- net /GND_Gaz: track 0.00 -> 25.1 mm
- net /RX: track 0.00 -> 15.6 mm
- net Net-(Q1-Pad1): track 0.00 -> 12.4 mm
- net Net-(IC1-Pad2): track 0.00 -> 9.72 mm
Other:
- board text added: "Back CU"

Commit message: maj
Parts:
- moved R4 20.5 mm to (121.2, 109.9)
- moved U1 20.1 mm to (142.7, 98.4)
- moved R5 14.3 mm to (119.9, 98.5)
- moved R6 13.3 mm to (119.9, 103.5)
- moved Rd4 6.74 mm to (158.0, 116.2)
Routing:
- net +5V: track 166.8 -> 108.8 mm
- net /GATE: track 0.00 -> 52.9 mm, vias 0 -> 2
- net +3V3: track 42.0 -> 88.5 mm
- net Net-(Ral1-Pad2): track 0.00 -> 46.0 mm, vias 0 -> 1
- net Net-(IC1-Pad3): track 99.2 -> 54.6 mm, vias 0 -> 3
- net /DATA_Sensor: track 0.00 -> 42.1 mm
- net Net-(Rd1-Pad1): track 0.00 -> 41.5 mm
- net /RX: track 15.6 -> 54.8 mm, vias 0 -> 4
- net Net-(Cd2-Pad1): track 70.3 -> 58.2 mm
- net Net-(Cd2-Pad2): track 65.2 -> 53.2 mm
- net Net-(C1-Pad2): track 56.4 -> 47.9 mm
- net Net-(Q1-Pad1): track 12.4 -> 19.9 mm
- net /TX: track 61.5 -> 66.5 mm, vias 1 -> 2
- net /RST: track 52.8 -> 57.7 mm
- net /GND_Gaz: track 25.1 -> 22.2 mm
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